File: Hardware/NES Module/NES Module.kicad_pcb (KiCad board)
At the start: 2 copper layers, 78.5 x 100 mm, 6 parts, among them J1 Conn_01x31, J2 Conn_01x31, J3 Conn_02x36_Top_Bottom

Commit message: edited nes module board
Connections:
- J2 pad 3: unconnected-(J2-Pin_3-Pad3) -> Net-(J2-Pin_3)
- J3 pad 38: unconnected-(J3-Pin_38-Pad38) -> Net-(J2-Pin_3)
Routing:
- net Net-(J2-Pin_3): track 0.00 -> 116.2 mm
- net GND: vias 3 -> 5
- net (no net): vias 1 -> 0
Changed lines of the file:
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@@
 	(net 55 "Net-(J2-Pin_20)")
 	(net 56 "unconnected-(J2-Pin_5-Pad5)")
-	(net 57 "unconnected-(J2-Pin_3-Pad3)")
+	(net 57 "Net-(J2-Pin_3)")
 	(net 58 "Net-(J2-Pin_26)")
 	(net 59 "Net-(J2-Pin_15)")
@@
 	(net 75 "unconnected-(J3-Pin_58-Pad58)")
 	(net 76 "unconnected-(J3-Pin_17-Pad17)")
-	(net 77 "unconnected-(J3-Pin_38-Pad38)")
-	(net 78 "unconnected-(J3-Pin_51-Pad51)")
-	(net 79 "unconnected-(J3-Pin_55-Pad55)")
-	(net 80 "unconnected-(J3-Pin_19-Pad19)")
-	(net 81 "unconnected-(J3-Pin_34-Pad34)")
-	(net 82 "unconnected-(J3-Pin_57-Pad57)")
-	(net 83 "unconnected-(J3-Pin_20-Pad20)")
+	(net 77 "unconnected-(J3-Pin_51-Pad51)")
+	(net 78 "unconnected-(J3-Pin_55-Pad55)")
+	(net 79 "unconnected-(J3-Pin_19-Pad19)")
+	(net 80 "unconnected-(J3-Pin_34-Pad34)")
+	(net 81 "unconnected-(J3-Pin_57-Pad57)")
+	(net 82 "unconnected-(J3-Pin_20-Pad20)")
 	(footprint "Resistor_THT:R_Axial_DIN0207_L6.3mm_D2.5mm_P10.16mm_Horizontal"
 		(layer "F.Cu")
@@
 			(layers "*.Cu" "*.Mask")
 			(remove_unused_layers no)
-			(net 57 "unconnected-(J2-Pin_3-Pad3)")
+			(net 57 "Net-(J2-Pin_3)")
 			(pinfunction "Pin_3")
 			(pintype "passive")
@@
 			(layers "*.Cu" "*.Mask")
 			(remove_unused_layers no)
-			(net 80 "unconnected-(J3-Pin_19-Pad19)")
+			(net 79 "unconnected-(J3-Pin_19-Pad19)")
 			(pinfunction "Pin_19")
 			(pintype "passive")
@@
 			(layers "*.Cu" "*.Mask")
 			(remove_unused_layers no)
-			(net 83 "unconnected-(J3-Pin_20-Pad20)")
+			(net 82 "unconnected-(J3-Pin_20-Pad20)")
 			(pinfunction "Pin_20")
 			(pintype "passive")
@@
 			(layers "*.Cu" "*.Mask")
 			(remove_unused_layers no)
-			(net 81 "unconnected-(J3-Pin_34-Pad34)")
+			(net 80 "unconnected-(J3-Pin_34-Pad34)")
 			(pinfunction "Pin_34")
 			(pintype "passive")
@@
 			(layers "*.Cu" "*.Mask")
 			(remove_unused_layers no)
-			(net 77 "unconnected-(J3-Pin_38-Pad38)")
+			(net 57 "Net-(J2-Pin_3)")
 			(pinfunction "Pin_38")
 			(pintype "passive")
@@
 			(layers "*.Cu" "*.Mask")
 			(remove_unused_layers no)
-			(net 78 "unconnected-(J3-Pin_51-Pad51)")
+			(net 77 "unconnected-(J3-Pin_51-Pad51)")
 			(pinfunction "Pin_51")
 			(pintype "passive")
@@
 			(layers "*.Cu" "*.Mask")
 			(remove_unused_layers no)
-			(net 79 "unconnected-(J3-Pin_55-Pad55)")
+			(net 78 "unconnected-(J3-Pin_55-Pad55)")
 			(pinfunction "Pin_55")
 			(pintype "passive")
@@
 			(layers "*.Cu" "*.Mask")
 			(remove_unused_layers no)
-			(net 82 "unconnected-(J3-Pin_57-Pad57)")
+			(net 81 "unconnected-(J3-Pin_57-Pad57)")
 			(pinfunction "Pin_57")
 			(pintype "passive")
@@
 	)
 	(via
-		(at 205 92)
+		(at 204 93.5)
 		(size 0.6)
 		(drill 0.3)
 		(layers "F.Cu" "B.Cu")
-		(net 0)
+		(free yes)
+		(net 1)
 	)
 	(via
@@
 	)
 	(via
+		(at 177.5 108.5)
+		(size 0.6)
+		(drill 0.3)
+		(layers "F.Cu" "B.Cu")
+		(free yes)
+		(net 1)
+	)
+	(via
 		(at 189.5 37.5)
 		(size 0.6)
@@
 	)
 	(segment
+		(start 171.5503 104.651)
+		(end 154.8163 121.385)
+		(width 0.2)
+		(layer "F.Cu")
+		(net 57)
+	)
+	(segment
+		(start 212.5 47.62)
+		(end 211.349 48.771)
+		(width 0.2)
+		(layer "F.Cu")
+		(net 57)
+	)
+	(segment
+		(start 211.349 48.771)
+		(end 211.349 62.83876)
+		(width 0.2)
+		(layer "F.Cu")
+		(net 57)
+	)
+	(segment
+		(start 210 64.18776)
+		(end 210 92.12776)
+		(width 0.2)
+		(layer "F.Cu")
+		(net 57)
+	)
+	(segment
+		(start 154.8163 121.385)
+		(end 151.415 121.385)
+		(width 0.2)
+		(layer "F.Cu")
+		(net 57)
+	)
+	(segment
+		(start 197.47676 104.651)
+		(end 171.5503 104.651)
+		(width 0.2)
+		(layer "F.Cu")
+		(net 57)
+	)
+	(segment
+		(start 210 92.12776)
+		(end 197.47676 104.651)
+		(width 0.2)
+		(layer "F.Cu")
+		(net 57)
+	)
+	(segment
+		(start 211.349 62.83876)
+		(end 210 64.18776)
+		(width 0.2)
+		(layer "F.Cu")
+		(net 57)
+	)
+	(segment
